Commit message: xacro updated

File: urdf/duo_robot.xacro (robot description, xacro)
@@ -8,8 +8,12 @@
   <xacro:property name="wheel_length" value="0.05"/>
   <xacro:property name="wheel_mass" value="0.1"/>
-  <xacro:property name="caster_wheel_radius" value="0.060"/>
+  <xacro:property name="caster_wheel_radius" value="0.050"/>
   <xacro:property name="caster_wheel_length" value="0.02"/>
   <xacro:property name="caster_mount_size" value="0.1 0.1 0.02"/>
-  <xacro:property name="caster_mount_mass" value="0.2"/>
+  <xacro:property name="caster_mount_mass" value="0.1"/>
+  <xacro:property name="dummy_mass" value="0.5"/>
+  <xacro:property name="dummy_ixx" value="0.02083333333333333"/>
+  <xacro:property name="dummy_iyy" value="0.010833333333333334"/>
+  <xacro:property name="dummy_izz" value="0.03083333333333333"/>
   <xacro:property name="green_color" value="0 1 0 1"/>
   <xacro:property name="black_color" value="0 0 0 1"/>
@@ -18,9 +22,4 @@
   <xacro:macro name="base_link" params="name length width height color">
     <link name="${name}">
-      <inertial>
-        <origin xyz="0 0 0" rpy="0 0 0"/>
-        <mass value="1.0"/>
-        <inertia ixx="0.02" ixy="0" ixz="0" iyy="0.02" iyz="0" izz="0.02"/>
-      </inertial>
       <visual>
         <geometry>
@@ -38,10 +37,10 @@
     </link>
   </xacro:macro>
-  <xacro:macro name="wheel_link" params="name radius length color mass">
+  <xacro:macro name="wheel_link" params="name radius length color mass ixx iyy izz">
     <link name="${name}">
       <inertial>
         <origin xyz="0 0 0" rpy="0 0 0"/>
         <mass value="${mass}"/>
-        <inertia ixx="0.001" ixy="0" ixz="0" iyy="0.001" iyz="0" izz="0.001"/>
+        <inertia ixx="${ixx}" ixy="0" ixz="0" iyy="${iyy}" iyz="0" izz="${izz}"/>
       </inertial>
       <visual>
@@ -60,12 +59,28 @@
     </link>
   </xacro:macro>
+  <!-- Base Reference Link -->
+  <link name="base_reference">
+    <inertial>
+      <origin xyz="0 0 0" rpy="0 0 0"/>
+      <mass value="0.001"/>
+      <inertia ixx="0.001" ixy="0" ixz="0" iyy="0.001" iyz="0" izz="0.001"/>
+    </inertial>
+  </link>
+  <!-- Dummy Link -->
+  <link name="dummy_link">
+    <inertial>
+      <origin xyz="0 0 0" rpy="0 0 0"/>
+      <mass value="${dummy_mass}"/>
+      <inertia ixx="${dummy_ixx}" ixy="0" ixz="0" iyy="${dummy_iyy}" iyz="0" izz="${dummy_izz}"/>
+    </inertial>
+  </link>
   <!-- Base Link -->
   <xacro:base_link name="base_link" length="${base_length}" width="${base_width}" height="${base_height}" color="${green_color}"/>
   <!-- Left Wheel -->
-  <xacro:wheel_link name="left_wheel" radius="${wheel_radius}" length="${wheel_length}" color="${black_color}" mass="${wheel_mass}"/>
+  <xacro:wheel_link name="left_wheel" radius="${wheel_radius}" length="${wheel_length}" color="${black_color}" mass="${wheel_mass}" ixx="0.0002708333333333334" iyy="0.0002708333333333334" izz="0.0005000000000000001"/>
   <!-- Right Wheel -->
-  <xacro:wheel_link name="right_wheel" radius="${wheel_radius}" length="${wheel_length}" color="${black_color}" mass="${wheel_mass}"/>
+  <xacro:wheel_link name="right_wheel" radius="${wheel_radius}" length="${wheel_length}" color="${black_color}" mass="${wheel_mass}" ixx="0.0002708333333333334" iyy="0.0002708333333333334" izz="0.0005000000000000001"/>
   <!-- Caster Wheel -->
-  <xacro:wheel_link name="caster_wheel" radius="${caster_wheel_radius}" length="${caster_wheel_length}" color="${black_color}" mass="0.05"/>
+  <xacro:wheel_link name="caster_wheel" radius="${caster_wheel_radius}" length="${caster_wheel_length}" color="${black_color}" mass="0.05" ixx="3.291666666666667e-05" iyy="3.291666666666667e-05" izz="6.250000000000001e-05"/>
   <!-- Caster Mount -->
   <link name="caster_mount">
@@ -73,5 +88,5 @@
       <origin xyz="0 0 0" rpy="0 0 0"/>
       <mass value="${caster_mount_mass}"/>
-      <inertia ixx="0.002" ixy="0" ixz="0" iyy="0.002" iyz="0" izz="0.002"/>
+      <inertia ixx="8.666666666666668e-05" ixy="0" ixz="0" iyy="8.666666666666668e-05" iyz="0" izz="0.00016666666666666672"/>
     </inertial>
     <visual>
@@ -85,8 +100,18 @@
   </link>
   <!-- Joint Definitions -->
+  <joint name="base_reference_to_base_link" type="fixed">
+    <parent link="base_reference" />
+    <child link="base_link" />
+    <origin xyz="0 0 0.17" rpy="0 0 0" /> <!-- Adjust the height here -->
+  </joint>
+  <joint name="base_link_to_dummy_link" type="fixed">
+    <parent link="base_link" />
+    <child link="dummy_link" />
+    <origin xyz="0 0 0" rpy="0 0 0" />
+  </joint>
   <joint name="left_wheel_joint" type="continuous">
     <parent link="base_link"/>
     <child link="left_wheel"/>
-    <origin xyz="-0.277 -0.07 -0.07" rpy="0 1.5708 0"/>
+    <origin xyz="-0.277 -0.13 -0.07" rpy="0 1.5708 0"/>
     <axis xyz="0 0 1"/>
   </joint>
@@ -94,5 +119,5 @@
     <parent link="base_link"/>
     <child link="right_wheel"/>
-    <origin xyz="0.277 -0.07 -0.07" rpy="0 1.5708 0"/>
+    <origin xyz="0.277 -0.13 -0.07" rpy="0 1.5708 0"/>
     <axis xyz="0 0 1"/>
   </joint>
@@ -100,5 +125,5 @@
     <parent link="base_link"/>
     <child link="caster_mount"/>
-    <origin xyz="0 0.25 -0.07" rpy="0 0 0"/>
+    <origin xyz="0 0.25 -0.062" rpy="0 0 0"/>
     <axis xyz="0 0 1"/>
   </joint>
@@ -106,5 +131,5 @@
     <parent link="caster_mount"/>
     <child link="caster_wheel"/>
-    <origin xyz="0 0 -0.03" rpy="0 1.5708 0"/>
+    <origin xyz="0 0 -0.06" rpy="0 1.5708 0"/>
     <axis xyz="0 0 1"/>
   </joint>
