Commit message: ultrasonic sensor added

File: urdf/duo.urdf (robot description, URDF)
Before this commit: robot duo, 7 links, 6 joints
Links:
- added link ultrasonic_sensor, mass 0.01; collision box size=0.046 0.02 0.021; visual box size=0.046 0.02 0.021
Joints:
- added joint ultrasonic_joint: type fixed, parent base_link, child ultrasonic_sensor, origin xyz=0 0.35 0.05 rpy=0 0 0
